File: uClouds_SE_Front_Panel.brd (EAGLE design)
At the start: 40.3 x 128.5 mm, 2 parts

Commit message: assembly process updates
Other:
- board text added: "µClouds SE Front Panel TD-UCSE-C-FP CC BY-SA 4.0 2019-02-18 tall-dog.com"
- board text removed: "µClouds SE Front Panel TD-UCSE-C-FP CC BY-SA 4.0 2018-05-20 tall-dog.com"
Changed lines of the file:
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@@
 <?xml version="1.0" encoding="utf-8"?>
 <!DOCTYPE eagle SYSTEM "eagle.dtd">
-<eagle version="9.0.1">
+<eagle version="9.3.1">
 <drawing>
 <settings>
@@
 TD-UCSE-C-FP
 CC BY-SA 4.0
-2018-05-20
+2019-02-18
 tall-dog.com</text>
 <text x="20.15" y="1.5" size="1.5" layer="30" ratio="10" rot="MR0" align="bottom-center">Panel
@@
 <param name="checkStop" value="0"/>
 <param name="checkValues" value="0"/>
+<param name="checkNames" value="1"/>
+<param name="checkWireStubs" value="1"/>
+<param name="checkPolygonWidth" value="0"/>
 <param name="useDiameter" value="13"/>
 <param name="maxErrors" value="50"/>
@@
 </autorouter>
 <elements>
-<element name="E$3" library="uClouds_SE_Library" package="NEG-OUT-L" value="" x="15.15" y="13.5"/>
-<element name="E$4" library="uClouds_SE_Library" package="NEG-OUT-R" value="" x="25.15" y="13.5"/>
+<element name="E$3" library="uClouds_SE_Library" package="NEG-OUT-L" value="" x="15.15" y="13.5" smashed="yes"/>
+<element name="E$4" library="uClouds_SE_Library" package="NEG-OUT-R" value="" x="25.15" y="13.5" smashed="yes"/>
 </elements>
 <signals>
@@
 </signal>
 </signals>
+<mfgpreviewcolors>
+<mfgpreviewcolor name="soldermaskcolor" color="0xC8008000"/>
+<mfgpreviewcolor name="silkscreencolor" color="0xFFFEFEFE"/>
+<mfgpreviewcolor name="backgroundcolor" color="0xFF282828"/>
+<mfgpreviewcolor name="coppercolor" color="0xFFFFBF00"/>
+<mfgpreviewcolor name="substratecolor" color="0xFF786E46"/>
+</mfgpreviewcolors>
 <errors>
 </errors>

Commit message: Updates for Revision D
Other:
- board text added: "Panel derived from work by Émilie Gillet of Mutable Instruments"
- board text added: "TD-UCSE-D"
- board text added: "µClouds SE Front Panel TD-UCSE-D-FP/B CC BY-SA 4.0 2019-12-13 tall-dog.com"
- board text removed: "Panel derived from work by Olivier Gillet of Mutable Instruments"
- board text removed: "TD-UCSE-C"
- board text removed: "µClouds SE Front Panel TD-UCSE-C-FP CC BY-SA 4.0 2019-02-18 tall-dog.com"
Changed lines of the file:
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@@
 <?xml version="1.0" encoding="utf-8"?>
 <!DOCTYPE eagle SYSTEM "eagle.dtd">
-<eagle version="9.3.1">
+<eagle version="9.5.2">
 <drawing>
 <settings>
@@
 <layers>
 <layer number="1" name="Top" color="4" fill="1" visible="yes" active="yes"/>
-<layer number="2" name="Route2" color="1" fill="3" visible="no" active="no"/>
-<layer number="15" name="Route15" color="4" fill="6" visible="no" active="no"/>
 <layer number="16" name="Bottom" color="1" fill="1" visible="yes" active="yes"/>
 <layer number="17" name="Pads" color="2" fill="1" visible="yes" active="yes"/>
@@
 <text x="20.15" y="127" size="1.5" layer="30" ratio="10" rot="MR0" align="top-center">µClouds SE
 Front Panel
-TD-UCSE-C-FP
+TD-UCSE-D-FP/B
 CC BY-SA 4.0
-2019-02-18
+2019-12-13
 tall-dog.com</text>
 <text x="20.15" y="1.5" size="1.5" layer="30" ratio="10" rot="MR0" align="bottom-center">Panel
 derived
 from work by
-Olivier Gillet
+Émilie Gillet
 of Mutable
 Instruments</text>
 <text x="20.15" y="120" size="1.5" layer="29" ratio="10" align="center">tall-dog.com</text>
-<text x="20.15" y="125.5" size="1.5" layer="29" ratio="10" align="center">TD-UCSE-C</text>
+<text x="20.15" y="125.5" size="1.5" layer="29" ratio="10" align="center">TD-UCSE-D</text>
 <wire x1="13.4" y1="127" x2="26.9" y2="127" width="0.15" layer="29"/>
 <wire x1="26.9" y1="127" x2="26.9" y2="124" width="0.15" layer="29"/>
