File: uClouds_SE_Control_Board.sch (EAGLE design)
At the start: 36 parts, among them J1 JACK-THONKICONN, J10 JACK-THONKICONN, J11 JACK-THONKICONN, J12 JACK-THONKICONN, J2 JACK-THONKICONN, J3 JACK-THONKICONN, J4 JACK-THONKICONN, J5 JACK-THONKICONN, J6 JACK-THONKICONN, J7 JACK-THONKICONN, J8 JACK-THONKICONN, J9 JACK-THONKICONN, P1 10k, P2 10k, P3 A50k, P4 10k, P5 10k, P6 10k, P7 10k

Commit message: Updates for Revision D
Connections:
- net -10V: now also P1.3, P2.3; no longer P1.1, P2.1
- net GND: now also P1.1, P2.1; no longer P1.3, P2.3
Other:
- note added: "D"
- note added: "Licensed: CC BY-SA 4.0 Board derived from work by Émilie Gillet of Mutable Instruments"
- note removed: "C"
- note removed: "Licensed: CC BY-SA 4.0 Board derived from work by Olivier Gillet of Mutable Instruments"
- moved on the sheet: P1, P2
