File: uClouds_SE_Assembly_Template.brd (EAGLE design)
At the start: 40 x 110.5 mm, 0 parts

Commit message: Updates for Revision D
Other:
- board text added: "2019-12-13"
- board text added: "TD-UCSE-D-AT"
- board text removed: "2019-02-18"
- board text removed: "TD-UCSE-B-AT"
Changed lines of the file:
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@@
 <?xml version="1.0" encoding="utf-8"?>
 <!DOCTYPE eagle SYSTEM "eagle.dtd">
-<eagle version="9.3.1">
+<eagle version="9.5.2">
 <drawing>
 <settings>
@@
 <layers>
 <layer number="1" name="Top" color="4" fill="1" visible="yes" active="yes"/>
-<layer number="2" name="Route2" color="1" fill="3" visible="no" active="no"/>
-<layer number="15" name="Route15" color="4" fill="6" visible="no" active="no"/>
 <layer number="16" name="Bottom" color="1" fill="1" visible="yes" active="yes"/>
 <layer number="17" name="Pads" color="2" fill="1" visible="yes" active="yes"/>
@@
 <hole x="7.5" y="31" drill="5.2"/>
 <text x="26.25" y="38.5" size="2" layer="21" rot="R90" align="center">Assembly Template</text>
-<text x="13.75" y="68.5" size="2" layer="21" rot="R90" align="center">TD-UCSE-B-AT</text>
-<text x="26.25" y="68.5" size="2" layer="21" rot="R90" align="center">2019-02-18</text>
+<text x="13.75" y="68.5" size="2" layer="21" rot="R90" align="center">TD-UCSE-D-AT</text>
+<text x="26.25" y="68.5" size="2" layer="21" rot="R90" align="center">2019-12-13</text>
 <text x="20" y="91" size="2.5" layer="21" ratio="10" rot="R180" align="center">THIS SIDE
 FACES UP</text>
 <text x="20" y="91" size="2" layer="22" ratio="10" rot="MR180" align="center">THIS SIDE
 FACES DOWN</text>
-<text x="26.25" y="68.5" size="2" layer="22" rot="MR90" align="center">TD-UCSE-B-AT</text>
-<text x="13.75" y="68.5" size="2" layer="22" rot="MR90" align="center">2019-02-18</text>
+<text x="26.25" y="68.5" size="2" layer="22" rot="MR90" align="center">TD-UCSE-D-AT</text>
+<text x="13.75" y="68.5" size="2" layer="22" rot="MR90" align="center">2019-12-13</text>
 <text x="26.25" y="38.5" size="2" layer="22" rot="MR90" align="center">µClouds SE</text>
 <text x="13.75" y="38.5" size="2" layer="22" rot="MR90" align="center">Assembly Template</text>

Commit message: Revision D
Parts:
- added E$1, E$2: (no value), uClouds_SE_Library:M2.5-HOLE
Routing:
- added copper zone on layer 1, net GND
- added copper zone on layer 16, net GND
Other:
- board text added: "2.0 mm"
- board text added: "2020-01-23 tall-dog.com"
- board text added: "µClouds SE Assembly Template"
- board text removed: "2019-12-13"
- board text removed: "Assembly Template"
- board text removed: "tall-dog.com"
- board text removed: "µClouds SE"
Changed lines of the file:
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@@
 <layers>
 <layer number="1" name="Top" color="4" fill="1" visible="yes" active="yes"/>
+<layer number="2" name="Route2" color="1" fill="3" visible="no" active="no"/>
+<layer number="15" name="Route15" color="4" fill="6" visible="no" active="no"/>
 <layer number="16" name="Bottom" color="1" fill="1" visible="yes" active="yes"/>
 <layer number="17" name="Pads" color="2" fill="1" visible="yes" active="yes"/>
@@
 <layer number="51" name="tDocu" color="7" fill="1" visible="yes" active="yes"/>
 <layer number="52" name="bDocu" color="7" fill="1" visible="yes" active="yes"/>
+<layer number="88" name="SimResults" color="9" fill="1" visible="no" active="no"/>
+<layer number="89" name="SimProbes" color="9" fill="1" visible="no" active="no"/>
+<layer number="90" name="Modules" color="5" fill="1" visible="no" active="no"/>
+<layer number="91" name="Nets" color="2" fill="1" visible="no" active="no"/>
+<layer number="92" name="Busses" color="1" fill="1" visible="no" active="no"/>
+<layer number="93" name="Pins" color="2" fill="1" visible="no" active="no"/>
+<layer number="94" name="Symbols" color="4" fill="1" visible="no" active="no"/>
+<layer number="95" name="Names" color="7" fill="1" visible="no" active="no"/>
+<layer number="96" name="Values" color="7" fill="1" visible="no" active="no"/>
+<layer number="97" name="Info" color="7" fill="1" visible="no" active="no"/>
+<layer number="98" name="Guide" color="6" fill="1" visible="no" active="no"/>
 </layers>
 <board>
@@
 <hole x="20" y="38.5" drill="6.2"/>
 <hole x="7.5" y="13" drill="3.2"/>
-<text x="13.75" y="38.5" size="2" layer="21" rot="R90" align="center">µClouds SE</text>
-<text x="20" y="17.5" size="2" layer="21" align="center">tall-dog.com</text>
+<text x="2" y="53.5" size="2" layer="21" ratio="12" rot="R90" align="center">µClouds SE Assembly Template</text>
+<text x="20" y="17.5" size="2" layer="21" ratio="12" align="center">TD-UCSE-D-AT</text>
 <hole x="32.5" y="31" drill="6.2"/>
 <hole x="20" y="23.5" drill="6.2"/>
@@
 <hole x="32.5" y="19.5" drill="3.2"/>
 <hole x="7.5" y="31" drill="5.2"/>
-<text x="26.25" y="38.5" size="2" layer="21" rot="R90" align="center">Assembly Template</text>
-<text x="13.75" y="68.5" size="2" layer="21" rot="R90" align="center">TD-UCSE-D-AT</text>
-<text x="26.25" y="68.5" size="2" layer="21" rot="R90" align="center">2019-12-13</text>
-<text x="20" y="91" size="2.5" layer="21" ratio="10" rot="R180" align="center">THIS SIDE
+<text x="38" y="53.5" size="2" layer="21" ratio="12" rot="R90" align="center">2020-01-23   tall-dog.com</text>
+<text x="20" y="91" size="2.5" layer="21" ratio="12" rot="R180" align="center">THIS SIDE
 FACES UP</text>
-<text x="20" y="91" size="2" layer="22" ratio="10" rot="MR180" align="center">THIS SIDE
+<text x="20" y="91" size="2" layer="22" ratio="12" rot="MR180" align="center">THIS SIDE
 FACES DOWN</text>
-<text x="26.25" y="68.5" size="2" layer="22" rot="MR90" align="center">TD-UCSE-D-AT</text>
-<text x="13.75" y="68.5" size="2" layer="22" rot="MR90" align="center">2019-12-13</text>
-<text x="26.25" y="38.5" size="2" layer="22" rot="MR90" align="center">µClouds SE</text>
-<text x="13.75" y="38.5" size="2" layer="22" rot="MR90" align="center">Assembly Template</text>
-<text x="20" y="17.5" size="2" layer="22" rot="MR0" align="center">tall-dog.com</text>
+<text x="20" y="17.5" size="2" layer="22" ratio="12" rot="MR0" align="center">TD-UCSE-D-AT</text>
+<text x="20" y="61" size="3.5" layer="22" ratio="12" rot="MR0" align="center">2.0 mm</text>
+<text x="20" y="61" size="3.5" layer="21" ratio="12" align="center">2.0 mm</text>
+<wire x1="12" y1="64" x2="28" y2="64" width="0.254" layer="21"/>
+<wire x1="28" y1="64" x2="28" y2="58" width="0.254" layer="21"/>
+<wire x1="28" y1="58" x2="12" y2="58" width="0.254" layer="21"/>
+<wire x1="12" y1="58" x2="12" y2="64" width="0.254" layer="21"/>
+<wire x1="12" y1="64" x2="28" y2="64" width="0.254" layer="22"/>
+<wire x1="28" y1="64" x2="28" y2="58" width="0.254" layer="22"/>
+<wire x1="28" y1="58" x2="12" y2="58" width="0.254" layer="22"/>
+<wire x1="12" y1="58" x2="12" y2="64" width="0.254" layer="22"/>
+<text x="38" y="53.5" size="2" layer="22" ratio="12" rot="MR90" align="center">µClouds SE Assembly Template</text>
+<text x="2" y="53.5" size="2" layer="22" ratio="12" rot="MR90" align="center">2020-01-23   tall-dog.com</text>
+<circle x="7.5" y="31" radius="4" width="0.25" layer="21"/>
+<circle x="7.5" y="31" radius="4" width="0.25" layer="22"/>
 </plain>
 <attributes>
@@
 </autorouter>
 <elements>
+<element name="E$1" library="uClouds_SE_Library" package="M2.5-HOLE" value="" x="20" y="107.5" smashed="yes"/>
+<element name="E$2" library="uClouds_SE_Library" package="M2.5-HOLE" value="" x="20" y="3" smashed="yes"/>
 </elements>
 <signals>
-<signal name="S$1">
-<via x="20" y="107.5" extent="1-16" drill="2.75" diameter="5"/>
-</signal>
-<signal name="S$2">
-<via x="20" y="3" extent="1-16" drill="2.75" diameter="5"/>
+<signal name="GND">
+<polygon width="0.5" layer="1" isolate="0.5">
+<vertex x="0" y="110.5"/>
+<vertex x="40" y="110.5"/>
+<vertex x="40" y="0"/>
+<vertex x="0" y="0"/>
+</polygon>
+<polygon width="0.5" layer="16" isolate="0.5">
+<vertex x="0" y="110.5"/>
+<vertex x="40" y="110.5"/>
+<vertex x="40" y="0"/>
+<vertex x="0" y="0"/>
+</polygon>
 </signal>
 </signals>
@@
 <mfgpreviewcolor name="substratecolor" color="0xFF786E46"/>
 </mfgpreviewcolors>
+<errors>
+</errors>
 </board>
 </drawing>
