File: uClouds_SE_Control_Board.brd (EAGLE design)
At the start: 40 x 110.5 mm, 38 parts, among them J1 JACK-THONKICONN, J10 JACK-THONKICONN, J11 JACK-THONKICONN, J12 JACK-THONKICONN, J2 JACK-THONKICONN, J3 JACK-THONKICONN, J4 JACK-THONKICONN, J5 JACK-THONKICONN, J6 JACK-THONKICONN, J7 JACK-THONKICONN, J8 JACK-THONKICONN, J9 JACK-THONKICONN, P1 10k, P2 10k, P3 A50k, P4 10k, P5 10k, P6 10k, P7 10k

Commit message: assembly process updates
Other:
- board text added: "2019-02-18"
- board text removed: "2018-06-06"
Changed lines of the file:
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@@
 <?xml version="1.0" encoding="utf-8"?>
 <!DOCTYPE eagle SYSTEM "eagle.dtd">
-<eagle version="9.0.1">
+<eagle version="9.3.1">
 <drawing>
 <settings>
@@
 <wire x1="37" y1="110.5" x2="40" y2="107.5" width="0" layer="20" curve="-90"/>
 <text x="1" y="87.5" size="2.5" layer="22" ratio="10" rot="MR180" align="center-left">TD-UCSE-C-CB</text>
-<text x="1" y="80" size="2.5" layer="22" ratio="10" rot="MR180" align="center-left">2018-06-06</text>
+<text x="1" y="80" size="2.5" layer="22" ratio="10" rot="MR180" align="center-left">2019-02-18</text>
 <text x="1" y="57.5" size="2.5" layer="22" ratio="10" rot="MR180" align="center-left">tall-dog.com</text>
 <text x="1" y="72.5" size="2.5" layer="22" ratio="10" rot="MR180" align="center-left">CC BY-SA 4.0</text>
@@
 <param name="checkStop" value="1"/>
 <param name="checkValues" value="0"/>
+<param name="checkNames" value="1"/>
+<param name="checkWireStubs" value="1"/>
+<param name="checkPolygonWidth" value="0"/>
 <param name="useDiameter" value="13"/>
 <param name="maxErrors" value="50"/>
@@
 <attribute name="NAME" x="25.25" y="104" size="1" layer="21" ratio="10" align="top-left"/>
 </element>
-<element name="HOLE2" library="uClouds_SE_Library" package="M2.5-HOLE" value="HOLE" x="20" y="3"/>
-<element name="HOLE1" library="uClouds_SE_Library" package="M2.5-HOLE" value="HOLE" x="20" y="107.5"/>
+<element name="HOLE2" library="uClouds_SE_Library" package="M2.5-HOLE" value="HOLE" x="20" y="3" smashed="yes"/>
+<element name="HOLE1" library="uClouds_SE_Library" package="M2.5-HOLE" value="HOLE" x="20" y="107.5" smashed="yes"/>
 <element name="H1" library="uClouds_SE_Library" package="PTH-0.1-2X5" value="HEADER-2X5-PTH-0.1" x="33" y="98.5" smashed="yes" rot="MR0">
 <attribute name="NAME" x="33" y="101.5" size="1" layer="22" ratio="10" rot="MR0" align="bottom-center"/>
@@
 <attribute name="NAME" x="35.5" y="13" size="1" layer="21" ratio="10" rot="R270" align="bottom-center"/>
 </element>
-<element name="U$1" library="uClouds_SE_Library" package="MARKING-CC-LOGO" value="" x="32.5" y="85.5" rot="MR0"/>
-<element name="U$2" library="uClouds_SE_Library" package="MARKING-OSH-LOGO-5MM" value="" x="32.5" y="56" rot="MR0"/>
+<element name="U$1" library="uClouds_SE_Library" package="MARKING-CC-LOGO" value="" x="32.5" y="85.5" smashed="yes" rot="MR0"/>
+<element name="U$2" library="uClouds_SE_Library" package="MARKING-OSH-LOGO-5MM" value="" x="32.5" y="56" smashed="yes" rot="MR0"/>
 <element name="P3" library="uClouds_SE_Library" package="POT-RK1109G" value="A50k" x="7.5" y="76" smashed="yes">
 <attribute name="NAME" x="7.5" y="83" size="1" layer="21" ratio="10" align="bottom-center"/>
@@
 </signal>
 </signals>
+<mfgpreviewcolors>
+<mfgpreviewcolor name="soldermaskcolor" color="0xC8008000"/>
+<mfgpreviewcolor name="silkscreencolor" color="0xFFFEFEFE"/>
+<mfgpreviewcolor name="backgroundcolor" color="0xFF282828"/>
+<mfgpreviewcolor name="coppercolor" color="0xFFFFBF00"/>
+<mfgpreviewcolor name="substratecolor" color="0xFF786E46"/>
+</mfgpreviewcolors>
 <errors>
 </errors>

Commit message: Updates for Revision D
Connections:
- net -10V: now also P1.P$3, P2.P$3; no longer P1.P$1, P2.P$1
- net GND: now also P1.P$1, P2.P$1; no longer P1.P$3, P2.P$3
Routing:
- net -10V: track 38.6 -> 36.7 mm
Other:
- board text added: "2019-12-09"
- board text added: "TD-UCSE-D-CB"
- board text added: "Émilie Gillet of Mutable Instruments"
- board text removed: "2019-02-18"
- board text removed: "Olivier Gillet of Mutable Instruments"
- board text removed: "TD-UCSE-C-CB"
Changed lines of the file:
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@@
 <?xml version="1.0" encoding="utf-8"?>
 <!DOCTYPE eagle SYSTEM "eagle.dtd">
-<eagle version="9.3.1">
+<eagle version="9.5.2">
 <drawing>
 <settings>
@@
 <setting verticaltext="up"/>
 </settings>
-<grid distance="0.25" unitdist="mm" unit="mm" style="lines" multiple="1" display="yes" altdistance="0.05" altunitdist="mm" altunit="mm"/>
+<grid distance="0.5" unitdist="mm" unit="mm" style="lines" multiple="1" display="yes" altdistance="0.05" altunitdist="mm" altunit="mm"/>
 <layers>
 <layer number="1" name="Top" color="4" fill="1" visible="yes" active="yes"/>
-<layer number="2" name="Route2" color="1" fill="3" visible="no" active="no"/>
-<layer number="15" name="Route15" color="4" fill="6" visible="no" active="no"/>
 <layer number="16" name="Bottom" color="1" fill="1" visible="yes" active="yes"/>
 <layer number="17" name="Pads" color="2" fill="1" visible="yes" active="yes"/>
@@
 <wire x1="40" y1="3" x2="37" y2="0" width="0" layer="20" curve="-90"/>
 <wire x1="37" y1="110.5" x2="40" y2="107.5" width="0" layer="20" curve="-90"/>
-<text x="1" y="87.5" size="2.5" layer="22" ratio="10" rot="MR180" align="center-left">TD-UCSE-C-CB</text>
-<text x="1" y="80" size="2.5" layer="22" ratio="10" rot="MR180" align="center-left">2019-02-18</text>
+<text x="1" y="87.5" size="2.5" layer="22" ratio="10" rot="MR180" align="center-left">TD-UCSE-D-CB</text>
+<text x="1" y="80" size="2.5" layer="22" ratio="10" rot="MR180" align="center-left">2019-12-09</text>
 <text x="1" y="57.5" size="2.5" layer="22" ratio="10" rot="MR180" align="center-left">tall-dog.com</text>
 <text x="1" y="72.5" size="2.5" layer="22" ratio="10" rot="MR180" align="center-left">CC BY-SA 4.0</text>
@@
 <text x="1" y="95" size="2.5" layer="22" ratio="10" rot="MR180" align="center-left">Control Board</text>
 <text x="20" y="10" size="1.35" layer="22" ratio="10" rot="MR0" align="center">Board derived from work by</text>
-<text x="20" y="8" size="1.35" layer="22" ratio="10" rot="MR0" align="center">Olivier Gillet of Mutable Instruments</text>
+<text x="20" y="8" size="1.35" layer="22" ratio="10" rot="MR0" align="center">Émilie Gillet of Mutable Instruments</text>
 <text x="32.5" y="80" size="1.4" layer="22" ratio="10" rot="MR180" align="center">BY-SA
 4.0</text>
@@
 <vertex x="0" y="0"/>
 </polygon>
-<contactref element="P1" pad="P$3"/>
-<contactref element="P2" pad="P$3"/>
 <contactref element="P7" pad="P$3"/>
 <contactref element="P4" pad="P$3"/>
@@
 <via x="5" y="77.75" extent="1-16" drill="0.35"/>
 <via x="7.5" y="85" extent="1-16" drill="0.35"/>
-<via x="19.5" y="83.5" extent="1-16" drill="0.35"/>
+<via x="20.5" y="84" extent="1-16" drill="0.35"/>
 <via x="28" y="84.5" extent="1-16" drill="0.35"/>
 <via x="37.5" y="83.5" extent="1-16" drill="0.35"/>
@@
 <via x="12" y="52.5" extent="1-16" drill="0.35"/>
 <via x="27.5" y="55" extent="1-16" drill="0.35"/>
-<via x="34" y="73.5" extent="1-16" drill="0.35"/>
+<via x="30.5" y="78" extent="1-16" drill="0.35"/>
 <via x="37" y="58.5" extent="1-16" drill="0.35"/>
 <via x="35.5" y="44.5" extent="1-16" drill="0.35"/>
@@
 <via x="13.5" y="82" extent="1-16" drill="0.35"/>
 <via x="27.5" y="71.5" extent="1-16" drill="0.35"/>
-<via x="29" y="73.5" extent="1-16" drill="0.35"/>
+<via x="31" y="73.5" extent="1-16" drill="0.35"/>
 <via x="28.5" y="81" extent="1-16" drill="0.35"/>
 <via x="23.5" y="81" extent="1-16" drill="0.35"/>
@@
 <via x="21.5" y="44.5" extent="1-16" drill="0.35"/>
 <via x="24" y="41.5" extent="1-16" drill="0.35"/>
-<via x="36.5" y="73" extent="1-16" drill="0.35"/>
+<via x="36" y="73.5" extent="1-16" drill="0.35"/>
 <via x="36.5" y="92.5" extent="1-16" drill="0.35"/>
 <via x="34.5" y="90" extent="1-16" drill="0.35"/>
@@
 <contactref element="H1" pad="5"/>
 <via x="19.5" y="100.5" extent="1-16" drill="0.35"/>
-<via x="22.5" y="74.5" extent="1-16" drill="0.35"/>
+<via x="24" y="75" extent="1-16" drill="0.35"/>
 <via x="21.5" y="64.5" extent="1-16" drill="0.35"/>
 <via x="23" y="63.5" extent="1-16" drill="0.35"/>
@@
 <via x="8.5" y="74.75" extent="1-16" drill="0.35"/>
 <via x="6.25" y="72.5" extent="1-16" drill="0.35"/>
+<contactref element="P1" pad="P$1"/>
+<contactref element="P2" pad="P$1"/>
 </signal>
 <signal name="A3V3">
@@
 </signal>
 <signal name="-10V">
-<contactref element="P1" pad="P$1"/>
-<contactref element="P2" pad="P$1"/>
 <contactref element="H2" pad="4"/>
-<wire x1="35.54" y1="69.77" x2="35.54" y2="77.46" width="0.25" layer="1"/>
-<wire x1="35.54" y1="77.46" x2="33.5" y2="79.5" width="0.25" layer="1"/>
-<wire x1="33.5" y1="79.5" x2="28" y2="79.5" width="0.25" layer="1"/>
-<wire x1="28" y1="79.5" x2="27" y2="78.5" width="0.25" layer="1"/>
-<wire x1="22.5" y1="76.5" x2="24.5" y2="78.5" width="0.25" layer="1"/>
-<wire x1="24.5" y1="78.5" x2="27" y2="78.5" width="0.25" layer="1"/>
-<wire x1="22.5" y1="76.5" x2="22.5" y2="81" width="0.25" layer="16"/>
-<wire x1="22.5" y1="81" x2="21.5" y2="82" width="0.25" layer="16"/>
-<wire x1="21.5" y1="82" x2="21.5" y2="85" width="0.25" layer="16"/>
-<wire x1="22.5" y1="91.5" x2="22.5" y2="86" width="0.25" layer="16"/>
-<wire x1="22.5" y1="86" x2="21.5" y2="85" width="0.25" layer="16"/>
+<contactref element="P1" pad="P$3"/>
+<contactref element="P2" pad="P$3"/>
+<wire x1="17.5" y1="91.5" x2="17.5" y2="86" width="0.25" layer="16"/>
+<wire x1="17.5" y1="81" x2="17.5" y2="76.5" width="0.25" layer="16"/>
+<wire x1="17.5" y1="76.5" x2="20.5" y2="73.5" width="0.25" layer="1"/>
+<wire x1="29" y1="73.5" x2="30.5" y2="72" width="0.25" layer="1"/>
+<wire x1="33.31" y1="72" x2="35.54" y2="69.77" width="0.25" layer="1"/>
+<wire x1="20.5" y1="73.5" x2="29" y2="73.5" width="0.25" layer="1"/>
+<wire x1="30.5" y1="72" x2="33.31" y2="72" width="0.25" layer="1"/>
+<wire x1="17.5" y1="86" x2="18.5" y2="85" width="0.25" layer="16"/>
+<wire x1="18.5" y1="82" x2="17.5" y2="81" width="0.25" layer="16"/>
+<wire x1="18.5" y1="85" x2="18.5" y2="82" width="0.25" layer="16"/>
 </signal>
 <signal name="IN-L-POT-A">
@@
 <signal name="IN-R-POT-A">
 <contactref element="H2" pad="8"/>
-<wire x1="8.5" y1="73" x2="27.23" y2="73" width="0.25" layer="1"/>
-<wire x1="30.46" y1="69.77" x2="27.23" y2="73" width="0.25" layer="1"/>
+<wire x1="8" y1="72.5" x2="27.73" y2="72.5" width="0.25" layer="1"/>
+<wire x1="30.46" y1="69.77" x2="27.73" y2="72.5" width="0.25" layer="1"/>
 <contactref element="P3" pad="1'"/>
 <wire x1="6.5" y1="66.3" x2="6.5" y2="71" width="0.25" layer="1"/>
-<wire x1="6.5" y1="71" x2="8.5" y2="73" width="0.25" layer="1"/>
+<wire x1="6.5" y1="71" x2="8" y2="72.5" width="0.25" layer="1"/>
 </signal>
 <signal name="IN-R-POT-B">

Commit message: Cleanup and silkscreen artwork updates
Parts:
- removed U$1: (no value), uClouds_SE_Library:MARKING-CC-LOGO
- removed U$2: (no value), uClouds_SE_Library:MARKING-OSH-LOGO-5MM
- H1, H2, H3, H4: device uClouds_SE_Library:PTH-0.1-2X5 -> uClouds_SE_Library:PTH-0.1-2X5-MALE
Other:
- board text added: "2019-12-18"
- board text removed: "2019-12-09"
- board text removed: "BY-SA 4.0"
- board text removed: "Board derived from work by"
- board text removed: "CC BY-SA 4.0"
- board text removed: "Control Board"
- board text removed: "open source hardware"
- board text removed: "tall-dog.com"
- board text removed: "µClouds SE"
- board text removed: "Émilie Gillet of Mutable Instruments"

Commit message: Revision D
Other:
- board text added: "2020-02-13"
- board text removed: "2019-12-18"
Changed lines of the file:
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@@
 <wire x1="37" y1="110.5" x2="40" y2="107.5" width="0.127" layer="20" curve="-90"/>
 <text x="20" y="87.5" size="2" layer="22" ratio="12" rot="MR180" align="center">TD-UCSE-D-CB</text>
-<text x="20" y="80" size="2" layer="22" ratio="12" rot="MR180" align="center">2019-12-18</text>
+<text x="20" y="80" size="2" layer="22" ratio="12" rot="MR180" align="center">2020-02-13</text>
 </plain>
 <attributes>
