File: uClouds_SE_Main_Board.brd (EAGLE design)
At the start: 40 x 110.5 mm, 142 parts, among them Q1 NPN-SOT23-BEC, Q2 NPN-SOT23-BEC, U1 STM32F405-LQFP-64, U10 ZENER-SOT-23, U2 WM8731-SSOP-28, U3 TL072-TSSOP-8, U4 MCP6004-TSSOP-14, U5 MCP6002-MSOP-8, U6 HC595, U7 TL072-TSSOP-8, U8 LM1117-SOT-223, U9 LM1117-SOT-223, X1 12.288MHz, X2 8MHz

Commit message: assembly process updates
Parts:
- added U$7: (no value), uClouds_SE_Library:TALL-DOG-LOGO-INVERT
Routing:
- net LED-1-GRN: track 25.3 -> 23.5 mm
- net N$20: track 7.08 -> 6.58 mm
Other:
- board text added: "2019-02-17"
- board text added: "TD-UCSE-C 2019-02-17 tall-dog.com"
- board text removed: "2018-06-06"
- board text removed: "TD-UCSE-C 2018-06-06 tall-dog.com"
Changed lines of the file:
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@@
 <?xml version="1.0" encoding="utf-8"?>
 <!DOCTYPE eagle SYSTEM "eagle.dtd">
-<eagle version="9.0.1">
+<eagle version="9.3.0">
 <drawing>
 <settings>
@@
 <setting verticaltext="up"/>
 </settings>
-<grid distance="0.25" unitdist="mm" unit="mm" style="lines" multiple="1" display="yes" altdistance="0.05" altunitdist="mm" altunit="mm"/>
+<grid distance="0.5" unitdist="mm" unit="mm" style="lines" multiple="1" display="yes" altdistance="0.05" altunitdist="mm" altunit="mm"/>
 <layers>
 <layer number="1" name="Top" color="4" fill="1" visible="yes" active="yes"/>
-<layer number="2" name="Route2" color="1" fill="3" visible="no" active="no"/>
-<layer number="15" name="Route15" color="4" fill="6" visible="no" active="no"/>
 <layer number="16" name="Bottom" color="1" fill="1" visible="yes" active="yes"/>
 <layer number="17" name="Pads" color="2" fill="1" visible="yes" active="yes"/>
@@
 <layer number="47" name="Measures" color="7" fill="1" visible="yes" active="yes"/>
 <layer number="48" name="Document" color="7" fill="1" visible="yes" active="yes"/>
+<layer number="49" name="Reference" color="7" fill="1" visible="yes" active="yes"/>
 <layer number="51" name="tDocu" color="7" fill="1" visible="yes" active="yes"/>
 <layer number="52" name="bDocu" color="7" fill="1" visible="yes" active="yes"/>
@@
 <wire x1="2.75" y1="91.25" x2="2.75" y2="106.25" width="0.127" layer="21"/>
 <wire x1="2.75" y1="106.25" x2="0.25" y2="106.25" width="0.127" layer="21"/>
-<text x="8" y="12" size="1.4" layer="21" ratio="10" align="center">2018-06-06</text>
+<text x="8" y="12" size="1.4" layer="21" ratio="10" align="center">2019-02-17</text>
 <wire x1="1" y1="10.75" x2="15" y2="10.75" width="0.127" layer="21"/>
 <wire x1="15" y1="10.75" x2="15" y2="13.25" width="0.127" layer="21"/>
 <wire x1="15" y1="13.25" x2="1" y2="13.25" width="0.127" layer="21"/>
 <wire x1="1" y1="13.25" x2="1" y2="10.75" width="0.127" layer="21"/>
-<text x="20" y="48" size="1.5" layer="22" ratio="10" rot="MR180" align="center">Board derived from
+<text x="35.5" y="53.5" size="1.4" layer="22" ratio="10" rot="SMR270" align="center">Board derived from
 work by Olivier Gillet of
 Mutable Instruments</text>
 <text x="15" y="21" size="2" layer="22" ratio="10" rot="MR0" align="center">TD-UCSE-C
-2018-06-06
+2019-02-17
 tall-dog.com</text>
 <rectangle x1="6" y1="11" x2="17" y2="15" layer="22"/>
@@
 <param name="checkStop" value="1"/>
 <param name="checkValues" value="0"/>
+<param name="checkNames" value="1"/>
+<param name="checkWireStubs" value="1"/>
+<param name="checkPolygonWidth" value="0"/>
 <param name="useDiameter" value="13"/>
 <param name="maxErrors" value="50"/>
@@
 </autorouter>
 <elements>
-<element name="HOLE1" library="uClouds_SE_Library" package="M2.5-HOLE" value="HOLE" x="20" y="107.5"/>
-<element name="HOLE2" library="uClouds_SE_Library" package="M2.5-HOLE" value="HOLE" x="20" y="3"/>
+<element name="HOLE1" library="uClouds_SE_Library" package="M2.5-HOLE" value="HOLE" x="20" y="107.5" smashed="yes"/>
+<element name="HOLE2" library="uClouds_SE_Library" package="M2.5-HOLE" value="HOLE" x="20" y="3" smashed="yes"/>
 <element name="H1" library="uClouds_SE_Library" package="PTH-0.1-2X5-FLIP" value="HEADER-2X5-PTH-0.1-FLIP" x="33" y="98.5" smashed="yes" rot="MR0">
 <attribute name="NAME" x="26.25" y="98.5" size="1" layer="21" ratio="10" rot="R270" align="top-center"/>
@@
 <attribute name="NAME" x="8" y="20.25" size="0.5" layer="51" ratio="10" rot="R180" align="center"/>
 </element>
-<element name="U$9" library="uClouds_SE_Library" package="FIDUCIAL" value="" x="27.5" y="105.5"/>
-<element name="U$1" library="uClouds_SE_Library" package="FIDUCIAL" value="" x="2" y="34"/>
-<element name="U$3" library="uClouds_SE_Library" package="FIDUCIAL" value="" x="37.5" y="2.5"/>
-<element name="U$2" library="uClouds_SE_Library" package="MARKING-OSH-LOGO-5MM" value="" x="18.5" y="34"/>
-<element name="U$6" library="uClouds_SE_Library" package="MARKING-CC-BY-SA-4.0" value="" x="38.5" y="20.5" rot="R90"/>
-<element name="U$4" library="uClouds_SE_Library" package="MARKING-CC-LOGO" value="" x="21" y="69"/>
-<element name="U$5" library="uClouds_SE_Library" package="MARKING-CC-LOGO" value="" x="25.25" y="78" rot="SMR90"/>
-<element name="U$8" library="uClouds_SE_Library" package="MARKING-OSH-LOGO-5MM" value="" x="25.25" y="88.5" rot="MR270"/>
+<element name="U$9" library="uClouds_SE_Library" package="FIDUCIAL" value="" x="27.5" y="105.5" smashed="yes"/>
+<element name="U$1" library="uClouds_SE_Library" package="FIDUCIAL" value="" x="2" y="34" smashed="yes"/>
+<element name="U$3" library="uClouds_SE_Library" package="FIDUCIAL" value="" x="37.5" y="2.5" smashed="yes"/>
+<element name="U$2" library="uClouds_SE_Library" package="MARKING-OSH-LOGO-5MM" value="" x="18.5" y="34" smashed="yes"/>
+<element name="U$6" library="uClouds_SE_Library" package="MARKING-CC-BY-SA-4.0" value="" x="38.5" y="20.5" smashed="yes" rot="R90"/>
+<element name="U$4" library="uClouds_SE_Library" package="MARKING-CC-LOGO" value="" x="21" y="69" smashed="yes"/>
+<element name="U$5" library="uClouds_SE_Library" package="MARKING-CC-LOGO" value="" x="25.25" y="78" smashed="yes" rot="SMR90"/>
+<element name="U$8" library="uClouds_SE_Library" package="MARKING-OSH-LOGO-5MM" value="" x="25.25" y="88.5" smashed="yes" rot="MR270"/>
+<element name="U$7" library="uClouds_SE_Library" package="TALL-DOG-LOGO-INVERT" value="" x="15" y="53.5" smashed="yes" rot="MR0"/>
 </elements>
 <signals>
@@
 <contactref element="R26" pad="2"/>
 <wire x1="10.5" y1="47.19" x2="8.5" y2="47.19" width="0.25" layer="1"/>
-<wire x1="6.3" y1="44" x2="6.8" y2="44" width="0.25" layer="1"/>
 <wire x1="6.3" y1="44" x2="6.3" y2="45.8" width="0.25" layer="1"/>
 <wire x1="6.3" y1="45.8" x2="7.69" y2="47.19" width="0.25" layer="1"/>
@@
 <wire x1="16.2" y1="79.75" x2="16.35" y2="79.6" width="0.25" layer="1"/>
 <via x="16.35" y="79.6" extent="1-16" drill="0.25"/>
-<wire x1="16.35" y1="79.6" x2="16.5" y2="79.45" width="0.25" layer="16"/>
 <wire x1="35.825" y1="51.3" x2="35.825" y2="53.475" width="0.25" layer="1"/>
 <wire x1="35.825" y1="53.475" x2="35.5" y2="53.8" width="0.25" layer="1"/>
@@
 <wire x1="15.25" y1="82.25" x2="16.4" y2="82.25" width="0.25" layer="1"/>
 <via x="16.4" y="82.25" extent="1-16" drill="0.25"/>
-<wire x1="16.4" y1="82.25" x2="16.5" y2="82.25" width="0.25" layer="16"/>
 <wire x1="35.54" y1="67.23" x2="35.54" y2="67.94" width="0.25" layer="16"/>
 <wire x1="35.54" y1="67.94" x2="36.8" y2="69.2" width="0.25" layer="16"/>
@@
 <contactref element="H3" pad="5"/>
 <contactref element="R40" pad="2"/>
-<wire x1="7" y1="37.23" x2="8.27" y2="38.5" width="0.25" layer="1"/>
 <wire x1="7" y1="37.23" x2="8.25" y2="38.48" width="0.25" layer="1"/>
 <wire x1="8.25" y1="38.48" x2="8.25" y2="40.3" width="0.25" layer="1"/>
@@
 </signal>
 </signals>
+<mfgpreviewcolors>
+<mfgpreviewcolor name="soldermaskcolor" color="0xC8008000"/>
+<mfgpreviewcolor name="silkscreencolor" color="0xFFFEFEFE"/>
+<mfgpreviewcolor name="backgroundcolor" color="0xFF282828"/>
+<mfgpreviewcolor name="coppercolor" color="0xFFFFBF00"/>
+<mfgpreviewcolor name="substratecolor" color="0xFF786E46"/>
+</mfgpreviewcolors>
 <errors>
 </errors>

Commit message: Updates for Revision D
Parts:
- removed S1, S2: SPST-EVQPA, uClouds_SE_Library:BUTTON-EVQPA
- removed U$9: (no value), uClouds_SE_Library:FIDUCIAL
- added C55: 0.1u, uClouds_SE_Library:0603-NP
- added R54: 470R, uClouds_SE_Library:0603-NP
- added U$101: (no value), uClouds_SE_Library:MARKING-CC-LOGO
- C1, C13, C20: value 10u -> 0.1u; device uClouds_SE_Library:ELECTRO-SMD-4.3MM -> uClouds_SE_Library:0603-NP
- C10: value 18p -> 2.2u
- C11, C36: value 18p -> 0.1u
- C12, C23: value 0.1u -> 18p
- C15, C2: value 1u -> 10u; device uClouds_SE_Library:0603-NP -> uClouds_SE_Library:ELECTRO-SMD-4.3MM
- C16: value 0.1u -> 1u
- C21, C27: value 18p -> 10u; device uClouds_SE_Library:0603-NP -> uClouds_SE_Library:ELECTRO-SMD-4.3MM
- C24: value 1u -> 0.1u
- C25: value 10u -> 1u; device uClouds_SE_Library:ELECTRO-SMD-4.3MM -> uClouds_SE_Library:0603-NP
- C28, C37: value 1n -> 18p
- C3: value 2.2u -> 1u
- C31: value 0.1u -> 1n
- C4: value 0.1u -> 10u; device uClouds_SE_Library:0603-NP -> uClouds_SE_Library:ELECTRO-SMD-4.3MM
- C40: value 10u -> 1n; device uClouds_SE_Library:ELECTRO-SMD-4.3MM -> uClouds_SE_Library:0603-NP
- C43: value 47u -> 10u; device uClouds_SE_Library:ELECTRO-SMD-6.6MM -> uClouds_SE_Library:ELECTRO-SMD-4.3MM
- C44: value 220p -> 47u; device uClouds_SE_Library:0603-NP -> uClouds_SE_Library:ELECTRO-SMD-6.6MM
- C46: value 0.1u -> 220p
- C47, C50, C53: value 47u -> 0.1u; device uClouds_SE_Library:ELECTRO-SMD-6.6MM -> uClouds_SE_Library:0603-NP
- C48, C52, C54: value 0.1u -> 47u; device uClouds_SE_Library:0603-NP -> uClouds_SE_Library:ELECTRO-SMD-6.6MM
- C5: value 10u -> 2.2u; device uClouds_SE_Library:ELECTRO-SMD-4.3MM -> uClouds_SE_Library:0603-NP
- C8: value 2.2u -> 18p
- H6: value HEADER-1X6-PTH-SHROUDED -> HEADER-1X2; device uClouds_SE_Library:JST-XH-6 -> uClouds_SE_Library:PTH-0.1-1X2
- R10: value 200k -> 180k
- R11: value 100k -> 200k
- R12, R20: value 10k -> 100k
- R13: value 33k -> 10k
- R14: value 47k -> 33k
- R15: value 66.5k -> 47k
- R16: value 5.6k -> 66.5k
- R17, R26: value 39k -> 5.6k
- R19: value 100k -> 39k
- R2: value 10k -> 100R
- R21: value 1k -> 10k
- R23: value 68R -> 1k
- R24: value 39k -> 68R
- R25: value 5.6k -> 39k
- R27: value 33k -> 39k
- R29: value 66.5k -> 33k
- R3: value 2.2k -> 100R
- R30: value 470R -> 66.5k
- R31: value 200k -> 470R
- R34: value 68R -> 200k
- R41: value 100k -> 68R
- R44: value 4.7R -> 100k; device uClouds_SE_Library:1206-NP -> uClouds_SE_Library:0603-NP
- R45: value 5.6k -> 4.7R; device uClouds_SE_Library:0603-NP -> uClouds_SE_Library:1206-NP
- R49: value 22k -> 5.6k
- R5: value 100k -> 2.2k
- R50: value 3.3k -> 22k
- R52: value 22k -> 3.3k
- R53: value 470R -> 22k
- R8: value 200k -> 100k
- R9: value 180k -> 200k
- U$2: device uClouds_SE_Library:MARKING-OSH-LOGO-5MM -> uClouds_SE_Library:MARKING-CC-LOGO
- U$4: device uClouds_SE_Library:MARKING-CC-LOGO -> uClouds_SE_Library:MARKING-OSH-LOGO-5MM
- U$5: device uClouds_SE_Library:MARKING-CC-LOGO -> uClouds_SE_Library:MARKING-CC-BY-SA-4.0
- U$6: device uClouds_SE_Library:MARKING-CC-BY-SA-4.0 -> uClouds_SE_Library:FIDUCIAL
- U1: value STM32F405-LQFP-64 -> WM8731-SSOP-28; device uClouds_SE_Library:LQFP-64 -> uClouds_SE_Library:SSOP-28
- U2: value WM8731-SSOP-28 -> STM32F405-LQFP-64; device uClouds_SE_Library:SSOP-28 -> uClouds_SE_Library:LQFP-64
- moved U$1 68.9 mm to (23.5, 99.5)
- moved U$5 59.0 mm to (38.5, 20.5), flipped to the top
- moved U$3 47.5 mm to (2.00, 34.0)
- moved U$2 35.1 mm to (21.0, 69.0)
- moved U$4 35.1 mm to (18.5, 34.0)
- moved C40 32.2 mm to (36.5, 48.0), turned to 0 degrees
- moved C31 31.9 mm to (36.5, 59.0)
- moved C44 31.3 mm to (33.8, 30.5)
- moved C10 30.4 mm to (3.00, 90.0)
- moved C8 30.4 mm to (33.2, 93.0)
- moved R2 30.1 mm to (5.50, 98.5)
- moved C20 28.6 mm to (2.25, 76.5), turned to 90 degrees
- moved R16 28.0 mm to (36.5, 61.0), turned to 0 degrees
- moved C21 27.8 mm to (30.8, 74.5)
- moved R1 25.7 mm to (5.50, 102.5), turned to 180 degrees
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- renumbered U$7 to U$100, U$8 to U$102
Connections:
- removed net BOOT: R2.2, S1.A1, S1.A2, U1.60
- removed net JTCK: H5.4, U1.49
- removed net JTDO: H5.6, U1.55
- removed net JTMS: H5.2, U1.46
- removed net N$35 (its old number): C41.C, C44.2, R45.2, R47.2
- new net JTCK/SWCLK: H5.4, U2.49
- new net JTDO/SWO: H5.6, U2.55
- new net JTMS/SWDIO: H5.2, U2.46
- new net N$19: C43.C, C46.2, R47.2, R49.2
- new net RX1: R3.2, U2.43
- new net TX1: R2.2, U2.42
- net -10V: now also C55.2, R10.1, R33.1, R54.1; no longer C54.2, R31.1, R53.1, R8.1
- net -12V: now also C33.1, C50.1, C52.C, R54.2; no longer C32.1, C49.1, C51.C, R53.2
- net 12V: now also C32.2, C44.A, C47.2, R45.1; no longer C31.2, C43.A, C46.2, R44.1
- net A3V3: now also C16.2, C19.2, C21.A, C25.2, C26.A, C35.2, C53.2, C54.A, U1.14, U1.8, U2.13; no longer C15.2, C17.2, C20.A, C23.2, C25.A, C33.2, C52.2, C53.A, U1.13, U2.14, U2.8
- net BLEND-CV: now also C29.2, R14.2, U2.21; no longer C28.2, R13.2, U1.21
- net BLEND-JACK: now also R6.1; no longer R5.1
- net BLEND-POT: now also U2.23; no longer U1.23
- net D3V3: now also C11.2, C14.2, C17.2, C2.A, C20.2, C3.2, C36.2, C4.A, C49.2, C51.A, R13.2, R21.2, R5.2, U1.1, U1.27, U2.19, U2.32, U2.48, U2.64; no longer C1.A, C12.2, C16.2, C19.2, C2.2, C35.2, C4.2, C48.2, C5.A, C50.A, R12.2, R20.2, R3.2, S1.B1, S1.B2, U1.19, U1.32, U1.48, U1.64, U2.1, U2.27
- net DENS-CV: now also C40.2, R30.2, U2.17; no longer C39.2, R29.2, U1.17
- net DENS-JACK: now also R44.1; no longer R43.1
- net DENS-POT: now also R34.1; no longer R33.1
- net FREEZE: now also R21.1, U2.59; no longer R20.1, U1.59
- net FREEZE-JACK: now also R20.1; no longer R19.1
- net GND: now also C1.1, C13.1, C15.C, C2.C, C20.1, C21.C, C23.2, C25.1, C26.C, C32.1, C33.2, C36.1, C4.C, C44.C, C47.1, C48.C, C49.1, C5.1, C50.2, C51.C, C52.A, C53.1, C54.C, C55.1, R18.1, R27.1, R47.1, U1.11, U1.15, U1.21, U1.22, U2.12, U2.18, U2.26, U2.60, U2.63; no longer C1.C, C13.C, C15.1, C2.1, C20.C, C21.2, C23.1, C25.C, C31.1, C32.2, C33.1, C4.1, C43.C, C44.1, C47.C, C48.1, C49.2, C5.C, C50.C, C51.A, C52.1, C53.C, C54.1, H6.1, R17.1, R2.1, R26.1, R45.1, S2.A1, S2.A2, U1.12, U1.18, U1.26, U1.63, U2.11, U2.15, U2.21, U2.22
- net I2C-SCL: now also R4.1, U1.24, U2.29; no longer R3.1, U1.29, U2.24
- net I2C-SDA: now also R5.1, U1.23, U2.30; no longer R4.1, U1.30, U2.23
- net I2S-LRCK: now also U1.5, U1.7, U2.33; no longer U1.33, U2.5, U2.7
- net I2S-SCK: now also U1.3, U2.34; no longer U1.34, U2.3
- net I2S-SIN: now also U1.6, U2.35; no longer U1.35, U2.6
- net I2S-SOUT: now also U1.4, U2.36; no longer U1.36, U2.4
- net IN-L: now also C43.A, U1.20; no longer C42.A, U2.20
- net IN-L-JACK: now also R53.1; no longer R52.1
- net IN-L-POT-A: now also R51.2; no longer R50.2
- net IN-L-POT-B: now also R49.1; no longer R48.1
- net IN-R: now also C42.A, U1.19; no longer C41.A, U2.19
- net IN-R-JACK: now also R50.1; no longer R49.1
- net IN-R-POT-A: now also R52.2; no longer R51.2
- net IN-R-POT-B: now also R48.1; no longer R47.1
- net JTDI: now also U2.50; no longer U1.50
- net LED-1-GRN: now also R41.2; no longer R40.2
- net LED-1-RED: now also R40.2; no longer R39.2
- net LED-2-GRN: now also R39.2; no longer R38.2
- net LED-2-RED: now also R38.2; no longer R37.2
- net LED-3-GRN: now also R37.2; no longer R36.2
- net LED-3-RED: now also R36.2; no longer R35.2
- net LED-4-GRN: now also R35.2; no longer R34.2
- net LED-4-RED: now also R24.2; no longer R23.2
- net LED-DATA: now also U2.57; no longer U1.57
- net LED-EN: now also U2.24; no longer U1.24
- net LED-FREEZE: now also R31.2; no longer R30.2
- net LED-SCK: now also U2.25; no longer U1.25
- net N$1: now also R24.1; no longer R23.1
- net N$10: now also R12.2; no longer R11.2
- net N$11: now also C22.1, U2.5; no longer C21.1, U1.5
- net N$12: now also C23.1, U2.6; no longer C22.1, U1.6
- net N$13: now also C31.1, R11.2, R16.1, R8.2; no longer C30.1, R10.2, R15.1, R7.2
- net N$14: now also C40.1, R30.1, R34.2, R44.2; no longer C39.1, R29.1, R33.2, R43.2
- net N$15: now also C38.1, R28.1, R32.2, R42.2; no longer C37.1, R27.1, R31.2, R41.2
- net N$16: now also C30.1, R10.2, R15.1, R7.2; no longer C29.1, R14.1, R6.2, R9.2
- net N$17: now also C39.1, R29.1, R33.2, R43.2; no longer C38.1, R28.1, R32.2, R42.2
- net N$18: now also C27.C, R17.1, R18.2; no longer C26.C, R16.1, R17.2
- net N$2: now also C48.A, R45.2; no longer C47.A, R44.2
- net N$20: now also C41.C, R26.1, R27.2; no longer C40.C, R25.1, R26.2
- net N$21: now also R20.2; no longer R19.2
- net N$22: now also C12.2, U1.25; no longer C11.2, U2.25
- net N$23: now also C8.2, U1.26; no longer C10.2, U2.26
- net N$24: now also C28.1, R17.2, R19.1; no longer C27.1, R16.2, R18.1
- net N$25: now also C28.2, R19.2, R22.1; no longer C27.2, R18.2, R21.1
- net N$26: now also C37.1, R25.1, R26.2; no longer C36.1, R24.1, R25.2
- net N$27: now also C13.2, C15.A, U1.16; no longer C13.A, C14.2, U2.16
- net N$28: now also R37.1; no longer R36.1
- net N$29: now also C37.2, R23.1, R25.2; no longer C36.2, R22.1, R24.2
- net N$3: now also R50.2, R52.1; no longer R49.2, R51.1
- net N$30: now also R38.1; no longer R37.1
- net N$31: now also R39.1; no longer R38.1
- net N$32: now also R40.1; no longer R39.1
- net N$33: now also R41.1; no longer R40.1
- net N$37: now also R31.1, U2.62; no longer R30.1, U1.62
- net N$4: now also R51.1, R53.2; no longer R50.1, R52.2
- net N$5: now also C29.1, R14.1, R6.2, R9.2; no longer C28.1, R13.1, R5.2, R8.2
- net N$6: now also R35.1; no longer R34.1
- net N$7: now also C5.2, U2.31; no longer C3.2, U1.31
- net N$8: now also C10.2, U2.47; no longer C8.2, U1.47
- net N$9: now also R36.1; no longer R35.1
- net OUT-L: now also C27.A, U1.12; no longer C26.A, U2.12
- net OUT-L-JACK: now also R22.2; no longer R21.2
- net OUT-R: now also C41.A, U1.13; no longer C40.A, U2.13
- net OUT-R-JACK: now also R23.2; no longer R22.2
- net PITCH-CV: now also C30.2, R15.2, U2.20; no longer C29.2, R14.2, U1.20
- net PITCH-JACK: now also R7.1; no longer R6.1
- net PITCH-POT: now also U2.9; no longer U1.9
- net POS-CV: now also C31.2, R16.2, U2.16; no longer C30.2, R15.2, U1.16
- net POS-JACK: now also R8.1; no longer R7.1
- net POS-POT: now also R11.1; no longer R10.1
- net RESET: now also C1.2, U2.7; no longer S2.B1, S2.B2, U1.7
- net RX: now also H6.2, R3.1; no longer H6.4, U1.43
- net SIZE-CV: now also C38.2, R28.2, U2.15; no longer C37.2, R27.2, U1.15
- net SIZE-JACK: now also R42.1; no longer R41.1
- net SIZE-POT: now also U2.8; no longer U1.8
- net SW-FREEZE: now also U2.61; no longer U1.61
- net SW-MEM: now also U2.51; no longer U1.51
- net SW-MODE: now also U2.52; no longer U1.52
- net TEXT-CV: now also C39.2, R29.2, U2.14; no longer C38.2, R28.2, U1.14
- net TEXT-JACK: now also R43.1; no longer R42.1
- net TEXT-POT: now also U2.22; no longer U1.22
- net TRIG: now also R13.1, U2.58; no longer R12.1, U1.58
- net TRIG-JACK: now also R12.1; no longer R11.1
- net TX: now also H6.1, R2.1; no longer H6.5, U1.42
Routing:
- net BOOT: track 57.1 -> 0.00 mm, vias 1 -> 0
- net JTDO/SWO: track 0.00 -> 24.8 mm, vias 0 -> 1
- net JTCK/SWCLK: track 0.00 -> 23.8 mm, vias 0 -> 1
- net JTCK: track 22.7 -> 0.00 mm, vias 1 -> 0
- net JTDO: track 22.5 -> 0.00 mm, vias 1 -> 0
- net JTMS/SWDIO: track 0.00 -> 19.0 mm, vias 0 -> 1
- net JTMS: track 18.9 -> 0.00 mm, vias 1 -> 0
- net RESET: track 54.0 -> 37.9 mm, vias 1 -> 2
- net TX1: track 0.00 -> 13.4 mm, vias 0 -> 2
- net RX1: track 0.00 -> 9.53 mm, vias 0 -> 2
- net RX: track 11.5 -> 2.80 mm, vias 1 -> 0
- net TX: track 11.3 -> 2.80 mm, vias 1 -> 0
- net N$35 (its old number): track 8.46 -> 0.00 mm
- net N$19: track 0.00 -> 8.46 mm
- net D3V3: track 217.6 -> 209.2 mm
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Other:
- board text added: "2019-12-09"
- board text added: "Board derived from work by Émilie Gillet of Mutable Instruments"
- board text added: "MAIN BOARD"
- board text added: "RX"
- board text added: "SWD/JTAG"
- board text added: "TD-UCSE-D 2019-12-09 tall-dog.com"
- board text added: "TD-UCSE-D-MB"
- board text added: "TX"
- board text added: "tall-dog.com"
- board text removed: "2019-02-17"
- board text removed: "BOOT"
- board text removed: "Board derived from work by Olivier Gillet of Mutable Instruments"
- board text removed: "FTDI"
- board text removed: "JTAG"
- board text removed: "RESET"
- board text removed: "TALL-DOG.COM"
- board text removed: "TD-UCSE-C 2019-02-17 tall-dog.com"
- board text removed: "TD-UCSE-C-MB"
- board text removed: "µClouds_SE"

Commit message: Cleanup and silkscreen artwork updates
Parts:
- removed U$100: (no value), uClouds_SE_Library:TALL-DOG-LOGO-INVERT
- removed U$101: (no value), uClouds_SE_Library:MARKING-CC-LOGO
- removed U$102: (no value), uClouds_SE_Library:MARKING-OSH-LOGO-5MM
- added U$10: (no value), uClouds_SE_Library:LOGO-PN
- added U$11: (no value), uClouds_SE_Library:LOGO-QC
- added U$7: (no value), uClouds_SE_Library:LOGO-REV
- added U$8: (no value), uClouds_SE_Library:LOGO-SN
- added U$9: (no value), uClouds_SE_Library:LOGO-TD
- H1, H2, H3, H4: device uClouds_SE_Library:PTH-0.1-2X5-FLIP -> uClouds_SE_Library:PTH-0.1-2X5-FEMALE
- U$2: device uClouds_SE_Library:MARKING-CC-LOGO -> uClouds_SE_Library:LOGO-OSHW
- U$4: device uClouds_SE_Library:MARKING-OSH-LOGO-5MM -> uClouds_SE_Library:LOGO-OSH
- U$5: device uClouds_SE_Library:MARKING-CC-BY-SA-4.0 -> uClouds_SE_Library:LOGO-CC
- moved U$5 65.8 mm to (15.0, 82.0), flipped to the bottom, turned to 0 degrees
- moved U$4 60.1 mm to (15.0, 94.0), flipped to the bottom
- moved U$2 6.71 mm to (15.0, 72.0), flipped to the bottom
Other:
- board text added: "TD-UCSE-D-MB 2019-12-18"
- board text removed: "2019-12-09"
- board text removed: "BY-SA 4.0"
- board text removed: "MAIN BOARD"
- board text removed: "SN"
- board text removed: "TD-UCSE-D 2019-12-09 tall-dog.com"
- board text removed: "TD-UCSE-D-MB"
- board text removed: "open source hardware"
- board text removed: "tall-dog.com"
- board text removed: "µClouds SE"
