File: uClouds_SE_Main_Board.sch (EAGLE design)
At the start: 134 parts, among them Q1 NPN-SOT23-BEC, Q2 NPN-SOT23-BEC, U1 STM32F405-LQFP-64, U10 ZENER-SOT-23, U2 WM8731-SSOP-28, U3 TL072-TSSOP-8, U4 MCP6004-TSSOP-14, U5 MCP6002-MSOP-8, U6 HC595, U7 TL072-TSSOP-8, U8 LM1117-SOT-223, U9 LM1117-SOT-223, X1 12.288MHz, X2 8MHz

Commit message: Updates for Revision D
Parts:
- removed S1, S2: SPST-EVQPA, uClouds_SE_Library:SPST-EVQPA
- added C55: 0.1u, uClouds_SE_Library:CAP-NP-0603
- added R54: 470R, uClouds_SE_Library:RESISTOR-0603
- C1, C13, C20: value 10u -> 0.1u; device uClouds_SE_Library:CAP-P-4.3MM -> uClouds_SE_Library:CAP-NP-0603
- C10: value 18p -> 2.2u
- C11, C36: value 18p -> 0.1u
- C12, C23: value 0.1u -> 18p
- C15, C2: value 1u -> 10u; device uClouds_SE_Library:CAP-NP-0603 -> uClouds_SE_Library:CAP-P-4.3MM
- C16: value 0.1u -> 1u
- C21, C27: value 18p -> 10u; device uClouds_SE_Library:CAP-NP-0603 -> uClouds_SE_Library:CAP-P-4.3MM
- C24: value 1u -> 0.1u
- C25: value 10u -> 1u; device uClouds_SE_Library:CAP-P-4.3MM -> uClouds_SE_Library:CAP-NP-0603
- C28, C37: value 1n -> 18p
- C3: value 2.2u -> 1u
- C31: value 0.1u -> 1n
- C4: value 0.1u -> 10u; device uClouds_SE_Library:CAP-NP-0603 -> uClouds_SE_Library:CAP-P-4.3MM
- C40: value 10u -> 1n; device uClouds_SE_Library:CAP-P-4.3MM -> uClouds_SE_Library:CAP-NP-0603
- C43: value 47u -> 10u; device uClouds_SE_Library:CAP-P-6.6MM -> uClouds_SE_Library:CAP-P-4.3MM
- C44: value 220p -> 47u; device uClouds_SE_Library:CAP-NP-0603 -> uClouds_SE_Library:CAP-P-6.6MM
- C46: value 0.1u -> 220p
- C47, C50, C53: value 47u -> 0.1u; device uClouds_SE_Library:CAP-P-6.6MM -> uClouds_SE_Library:CAP-NP-0603
- C48, C52, C54: value 0.1u -> 47u; device uClouds_SE_Library:CAP-NP-0603 -> uClouds_SE_Library:CAP-P-6.6MM
- C5: value 10u -> 2.2u; device uClouds_SE_Library:CAP-P-4.3MM -> uClouds_SE_Library:CAP-NP-0603
- C8: value 2.2u -> 18p
- H6: value HEADER-1X6-PTH-SHROUDED -> HEADER-1X2; device uClouds_SE_Library:HEADER-1X6-PTH-SHROUDED -> uClouds_SE_Library:HEADER-1X2
- R10: value 200k -> 180k
- R11: value 100k -> 200k
- R12, R20: value 10k -> 100k
- R13: value 33k -> 10k
- R14: value 47k -> 33k
- R15: value 66.5k -> 47k
- R16: value 5.6k -> 66.5k
- R17, R26: value 39k -> 5.6k
- R19: value 100k -> 39k
- R2: value 10k -> 100R
- R21: value 1k -> 10k
- R23: value 68R -> 1k
- R24: value 39k -> 68R
- R25: value 5.6k -> 39k
- R27: value 33k -> 39k
- R29: value 66.5k -> 33k
- R3: value 2.2k -> 100R
- R30: value 470R -> 66.5k
- R31: value 200k -> 470R
- R34: value 68R -> 200k
- R41: value 100k -> 68R
- R44: value 4.7R -> 100k; device uClouds_SE_Library:RESISTOR-1206 -> uClouds_SE_Library:RESISTOR-0603
- R45: value 5.6k -> 4.7R; device uClouds_SE_Library:RESISTOR-0603 -> uClouds_SE_Library:RESISTOR-1206
- R49: value 22k -> 5.6k
- R5: value 100k -> 2.2k
- R50: value 3.3k -> 22k
- R52: value 22k -> 3.3k
- R53: value 470R -> 22k
- R8: value 200k -> 100k
- R9: value 180k -> 200k
- U1: value STM32F405-LQFP-64 -> WM8731-SSOP-28; device uClouds_SE_Library:STM32F405-LQFP-64 -> uClouds_SE_Library:WM8731-SSOP-28
- U2: value WM8731-SSOP-28 -> STM32F405-LQFP-64; device uClouds_SE_Library:WM8731-SSOP-28 -> uClouds_SE_Library:STM32F405-LQFP-64
Connections:
- removed net BOOT: R2.2, S1.1, U1.BOOT0
- removed net JTCK: H5.4, U1.PA14
- removed net JTDO: H5.6, U1.PB3
- removed net JTMS: H5.2, U1.PA13
- removed net N$35 (its old number): C41.NEG, C44.2, R45.2, R47.2
- new net JTCK/SWCLK: H5.4, U2.PA14
- new net JTDO/SWO: H5.6, U2.PB3
- new net JTMS/SWDIO: H5.2, U2.PA13
- new net N$19: C43.NEG, C46.2, R47.2, R49.2
- new net RX1: R3.2, U2.PA10
- new net TX1: R2.2, U2.PA9
- net -10V: now also C55.2, R10.1, R33.1, R54.1; no longer C54.2, R31.1, R53.1, R8.1
- net -12V: now also C33.1, C50.1, C52.NEG, R54.2; no longer C32.1, C49.1, C51.NEG, R53.2
- net 12V: now also C32.2, C44.POS, C47.2, R45.1; no longer C31.2, C43.POS, C46.2, R44.1
- net A3V3: now also C16.2, C19.2, C21.POS, C25.2, C26.POS, C35.2, C53.2, C54.POS, U1.AVDD, U1.HPVDD, U2.VDDA; no longer C15.2, C17.2, C20.POS, C23.2, C25.POS, C33.2, C52.2, C53.POS, U1.VDDA, U2.AVDD, U2.HPVDD
- net BLEND-CV: now also C29.2, R14.2, U2.PA5; no longer C28.2, R13.2, U1.PA5
- net BLEND-JACK: now also R6.1; no longer R5.1
- net BLEND-POT: now also U2.PA7; no longer U1.PA7
- net D3V3: now also C11.2, C14.2, C17.2, C2.POS, C20.2, C3.2, C36.2, C4.POS, C49.2, C51.POS, R13.2, R21.2, R5.2, U1.DBVDD, U1.DCVDD, U2.VDD1, U2.VDD2, U2.VDD3, U2.VDD4; no longer C1.POS, C12.2, C16.2, C19.2, C2.2, C35.2, C4.2, C48.2, C5.POS, C50.POS, R12.2, R20.2, R3.2, S1.2, U1.VDD1, U1.VDD2, U1.VDD3, U1.VDD4, U2.DBVDD, U2.DCVDD
- net DENS-CV: now also C40.2, R30.2, U2.PA3; no longer C39.2, R29.2, U1.PA3
- net DENS-JACK: now also R44.1; no longer R43.1
- net DENS-POT: now also R34.1; no longer R33.1
- net FREEZE: now also R21.1, U2.PB7; no longer R20.1, U1.PB7
- net FREEZE-JACK: now also R20.1; no longer R19.1
- net GND: now also C1.1, C13.1, C15.NEG, C2.NEG, C20.1, C21.NEG, C23.2, C25.1, C26.NEG, C32.1, C33.2, C36.1, C4.NEG, C44.NEG, C47.1, C48.NEG, C49.1, C5.1, C50.2, C51.NEG, C52.POS, C53.1, C54.NEG, C55.1, R18.1, R27.1, R47.1, U1.AGND, U1.CSB, U1.DGND, U1.HPGND, U1.MODE, U2.BOOT0, U2.PB0, U2.PB2, U2.VSS3, U2.VSS4, U2.VSSA; no longer C1.NEG, C13.NEG, C15.1, C2.1, C20.NEG, C21.2, C23.1, C25.NEG, C31.1, C32.2, C33.1, C4.1, C43.NEG, C44.1, C47.NEG, C48.1, C49.2, C5.NEG, C50.NEG, C51.POS, C52.1, C53.NEG, C54.1, H6.1, R17.1, R2.1, R26.1, R45.1, S2.1, U1.PB0, U1.PB2, U1.VSS3, U1.VSS4, U1.VSSA, U2.AGND, U2.CSB, U2.DGND, U2.HPGND, U2.MODE
- net I2C-SCL: now also R4.1, U1.SCLK, U2.PB10; no longer R3.1, U1.PB10, U2.SCLK
- net I2C-SDA: now also R5.1, U1.SDIN, U2.PB11; no longer R4.1, U1.PB11, U2.SDIN
- net I2S-LRCK: now also U1.ADCLRC, U1.DACLRC, U2.PB12; no longer U1.PB12, U2.ADCLRC, U2.DACLRC
- net I2S-SCK: now also U1.BCLK, U2.PB13; no longer U1.PB13, U2.BCLK
- net I2S-SIN: now also U1.ADCDAT, U2.PB14; no longer U1.PB14, U2.ADCDAT
- net I2S-SOUT: now also U1.DACDAT, U2.PB15; no longer U1.PB15, U2.DACDAT
- net IN-L: now also C43.POS, U1.LLINEIN; no longer C42.POS, U2.LLINEIN
- net IN-L-JACK: now also R53.1; no longer R52.1
- net IN-L-POT-A: now also R51.2; no longer R50.2
- net IN-L-POT-B: now also R49.1; no longer R48.1
- net IN-R: now also C42.POS, U1.RLINEIN; no longer C41.POS, U2.RLINEIN
- net IN-R-JACK: now also R50.1; no longer R49.1
- net IN-R-POT-A: now also R52.2; no longer R51.2
- net IN-R-POT-B: now also R48.1; no longer R47.1
- net JTDI: now also U2.PA15; no longer U1.PA15
- net LED-1-GRN: now also R41.2; no longer R40.2
- net LED-1-RED: now also R40.2; no longer R39.2
- net LED-2-GRN: now also R39.2; no longer R38.2
- net LED-2-RED: now also R38.2; no longer R37.2
- net LED-3-GRN: now also R37.2; no longer R36.2
- net LED-3-RED: now also R36.2; no longer R35.2
- net LED-4-GRN: now also R35.2; no longer R34.2
- net LED-4-RED: now also R24.2; no longer R23.2
- net LED-DATA: now also U2.PB5; no longer U1.PB5
- net LED-EN: now also U2.PC4; no longer U1.PC4
- net LED-FREEZE: now also R31.2; no longer R30.2
- net LED-SCK: now also U2.PC5; no longer U1.PC5
- net N$1: now also R24.1; no longer R23.1
- net N$10: now also R12.2; no longer R11.2
- net N$11: now also C22.1, U2.PD0; no longer C21.1, U1.PD0
- net N$12: now also C23.1, U2.PD1; no longer C22.1, U1.PD1
- net N$13: now also C31.1, R11.2, R16.1, R8.2; no longer C30.1, R10.2, R15.1, R7.2
- net N$14: now also C40.1, R30.1, R34.2, R44.2; no longer C39.1, R29.1, R33.2, R43.2
- net N$15: now also C38.1, R28.1, R32.2, R42.2; no longer C37.1, R27.1, R31.2, R41.2
- net N$16: now also C30.1, R10.2, R15.1, R7.2; no longer C29.1, R14.1, R6.2, R9.2
- net N$17: now also C39.1, R29.1, R33.2, R43.2; no longer C38.1, R28.1, R32.2, R42.2
- net N$18: now also C27.NEG, R17.1, R18.2; no longer C26.NEG, R16.1, R17.2
- net N$2: now also C48.POS, R45.2; no longer C47.POS, R44.2
- net N$20: now also C41.NEG, R26.1, R27.2; no longer C40.NEG, R25.1, R26.2
- net N$21: now also R20.2; no longer R19.2
- net N$22: now also C12.2, U1.XTI/MCLK; no longer C11.2, U2.XTI/MCLK
- net N$23: now also C8.2, U1.XTO; no longer C10.2, U2.XTO
- net N$24: now also C28.1, R17.2, R19.1; no longer C27.1, R16.2, R18.1
- net N$25: now also C28.2, R19.2, R22.1; no longer C27.2, R18.2, R21.1
- net N$26: now also C37.1, R25.1, R26.2; no longer C36.1, R24.1, R25.2
- net N$27: now also C13.2, C15.POS, U1.VMID; no longer C13.POS, C14.2, U2.VMID
- net N$28: now also R37.1; no longer R36.1
- net N$29: now also C37.2, R23.1, R25.2; no longer C36.2, R22.1, R24.2
- net N$3: now also R50.2, R52.1; no longer R49.2, R51.1
- net N$30: now also R38.1; no longer R37.1
- net N$31: now also R39.1; no longer R38.1
- net N$32: now also R40.1; no longer R39.1
- net N$33: now also R41.1; no longer R40.1
- net N$37: now also R31.1, U2.PB9; no longer R30.1, U1.PB9
- net N$4: now also R51.1, R53.2; no longer R50.1, R52.2
- net N$5: now also C29.1, R14.1, R6.2, R9.2; no longer C28.1, R13.1, R5.2, R8.2
- net N$6: now also R35.1; no longer R34.1
- net N$7: now also C5.2, U2.VSS1; no longer C3.2, U1.VSS1
- net N$8: now also C10.2, U2.VSS2; no longer C8.2, U1.VSS2
- net N$9: now also R36.1; no longer R35.1
- net OUT-L: now also C27.POS, U1.LOUT; no longer C26.POS, U2.LOUT
- net OUT-L-JACK: now also R22.2; no longer R21.2
- net OUT-R: now also C41.POS, U1.ROUT; no longer C40.POS, U2.ROUT
- net OUT-R-JACK: now also R23.2; no longer R22.2
- net PITCH-CV: now also C30.2, R15.2, U2.PA4; no longer C29.2, R14.2, U1.PA4
- net PITCH-JACK: now also R7.1; no longer R6.1
- net PITCH-POT: now also U2.PC1; no longer U1.PC1
- net POS-CV: now also C31.2, R16.2, U2.PA2; no longer C30.2, R15.2, U1.PA2
- net POS-JACK: now also R8.1; no longer R7.1
- net POS-POT: now also R11.1; no longer R10.1
- net RESET: now also C1.2, U2.NRST; no longer S2.2, U1.NRST
- net RX: now also H6.2, R3.1; no longer H6.4, U1.PA10
- net SIZE-CV: now also C38.2, R28.2, U2.PA1; no longer C37.2, R27.2, U1.PA1
- net SIZE-JACK: now also R42.1; no longer R41.1
- net SIZE-POT: now also U2.PC0; no longer U1.PC0
- net SW-FREEZE: now also U2.PB8; no longer U1.PB8
- net SW-MEM: now also U2.PC10; no longer U1.PC10
- net SW-MODE: now also U2.PC11; no longer U1.PC11
- net TEXT-CV: now also C39.2, R29.2, U2.PA0; no longer C38.2, R28.2, U1.PA0
- net TEXT-JACK: now also R43.1; no longer R42.1
- net TEXT-POT: now also U2.PA6; no longer U1.PA6
- net TRIG: now also R13.1, U2.PB6; no longer R12.1, U1.PB6
- net TRIG-JACK: now also R12.1; no longer R11.1
- net TX: now also H6.1, R2.1; no longer H6.5, U1.PA9
Other:
- note added: "D"
- note added: "Licensed: CC BY-SA 4.0 Board derived from work by Émilie Gillet of Mutable Instruments"
- note removed: "C"
- note removed: "Licensed: CC BY-SA 4.0 Board derived from work by Olivier Gillet of Mutable Instruments"
- moved on the sheet: C10, C11, C12, C14, C16, C17, C18, C19, C22, C23, C24, C29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
